File: KiCAD_Files/Driver_High.kicad_sch (KiCad schematic)
At the start: 25 parts, among them Q902 DMP3099-x, U902 FODM217A, U904 UCC21222DR

Commit message: Schematic close to completion.
Signed-off-by: Jean Alinei <jean.alinei@owntech.org>
Parts:
- renumbered C906 to C66, C908 to C67, C901 to C68, C910 to C69, C904 to C70, C911 to C71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
