File: KiCAD_Files/Feeder.kicad_sch (KiCad schematic)
At the start: 81 parts, among them J5001 B2B-EH-A(LF)(SN), J5002 B2B-EH-A(LF)(SN), J5003 Header_2_54_01x03, Q5001 DMN10H220L-7, Q5002 TK13P25D,RQ, T5001 PA2467NL, U5001 MCP6486UT-E/LT, U5002 AZ1117CH-5.0TRG1, U5003 NCP12700ADNR2G, U5004 AZ1117CH-5.0TRG1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

Commit message: Schematic close to completion.
Signed-off-by: Jean Alinei <jean.alinei@owntech.org>
Parts:
- renumbered C5002 to C10, C5003 to C15, C5005 to C16, C5006 to C17, C5008 to C20, C5009 to C21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
