File: KiCAD_Files/AC_voltage_sense.kicad_sch (KiCad schematic)
At the start: 19 parts, among them U501 AMC1301DWR, U502 MCP6486UT-E/LT

Commit message: Added TL431 for AC measurement 5V regulation. Added more film capacitance. Increased size of 100V ceramic caps to 1210.
Signed-off-by: Jean Alinei <jean.alinei@owntech.org>
Parts:
- U502: footprint Package_TO_SOT_SMD:SOT-353_SC-70-5_Handsoldering -> Package_TO_SOT_SMD:SOT-353_SC-70-5; symbol Symbols:MCP6486UT-E/LT -> Symbols:MCP6486UT-E/LT
Changed lines of the file:
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@@
 		(polyline
 			(pts
-				(xy 97.79 107.95) (xy 97.79 35.56) (xy 20.32 35.56) (xy 20.32 71.755) (xy 20.32 74.93) (xy 20.32 107.95)
+				(xy 97.79 107.95) (xy 97.79 35.56) (xy 30.48 35.56) (xy 30.48 74.93) (xy 20.32 74.93) (xy 20.32 107.95)
 			)
 			(stroke
@@
 	)
 	(symbol
-		(lib_id "Symbols:+12V_PGND")
+		(lib_id "power:+12V")
 		(at 170.18 46.99 0)
 		(unit 1)
 		(exclude_from_sim no)
-		(in_bom no)
-		(on_board no)
+		(in_bom yes)
+		(on_board yes)
 		(dnp no)
 		(fields_autoplaced yes)
@@
 		)
 		(property "Footprint" ""
-			(at 173.355 44.45 0)
+			(at 170.18 46.99 0)
 			(effects
 				(font
@@
 		)
 		(property "Datasheet" ""
-			(at 173.355 44.45 0)
-			(effects
-				(font
-					(size 1.27 1.27)
-				)
-				(hide yes)
-			)
-		)
-		(property "Description" ""
+			(at 170.18 46.99 0)
+			(effects
+				(font
+					(size 1.27 1.27)
+				)
+				(hide yes)
+			)
+		)
+		(property "Description" "Power symbol creates a global label with name \"+12V\""
 			(at 170.18 46.99 0)
 			(effects
@@
 	)
 	(symbol
-		(lib_id "Symbols:DGND")
+		(lib_id "power:GNDD")
 		(at 119.38 58.42 0)
 		(unit 1)
@@
 			)
 		)
-		(property "Description" ""
+		(property "Description" "Power symbol creates a global label with name \"GNDD\" , digital ground"
 			(at 119.38 58.42 0)
 			(effects
@@
 	)
 	(symbol
-		(lib_id "Symbols:MCP6486UT-E/LT ")
+		(lib_id "Symbols:MCP6486UT-E/LT")
 		(at 170.18 72.39 0)
 		(unit 1)
@@
 			)
 		)
-		(property "Footprint" "Package_TO_SOT_SMD:SOT-353_SC-70-5_Handsoldering"
+		(property "Footprint" "Package_TO_SOT_SMD:SOT-353_SC-70-5"
 			(at 175.26 78.74 0)
 			(effects
@@
 	)
 	(symbol
-		(lib_id "Symbols:+12V_PGND")
+		(lib_id "power:+12V")
 		(at 119.38 45.72 0)
 		(unit 1)
 		(exclude_from_sim no)
-		(in_bom no)
-		(on_board no)
+		(in_bom yes)
+		(on_board yes)
 		(dnp no)
 		(fields_autoplaced yes)
@@
 		)
 		(property "Footprint" ""
-			(at 122.555 43.18 0)
+			(at 119.38 45.72 0)
 			(effects
 				(font
@@
 		)
 		(property "Datasheet" ""
-			(at 122.555 43.18 0)
-			(effects
-				(font
-					(size 1.27 1.27)
-				)
-				(hide yes)
-			)
-		)
-		(property "Description" ""
 			(at 119.38 45.72 0)
 			(effects
@@
 			)
 		)
+		(property "Description" "Power symbol creates a global label with name \"+12V\""
+			(at 119.38 45.72 0)
+			(effects
+				(font
+					(size 1.27 1.27)
+				)
+				(hide yes)
+			)
+		)
 		(pin "1"
 		)
@@
 	)
 	(symbol
-		(lib_name "R_Small_14")
 		(lib_id "Device:R_Small")
 		(at 128.27 74.93 90)
@@
 			)
 		)
-		(property "Datasheet" "${KIPRJMOD}\\datasheet\\PYu_RT_1_to_0_01_RoHS_L_12-3003070.pdf"
+		(property "Datasheet" "~"
 			(at 128.27 74.93 0)
 			(effects
@@
 			)
 		)
-		(property "Description" ""
+		(property "Description" "Resistor, small symbol"
 			(at 128.27 74.93 0)
 			(effects
@@
 			)
 		)
-		(property "Description" ""
+		(property "Description" "Resistor, small symbol"
 			(at 68.58 77.47 0)
 			(effects
@@
 			)
 		)
-		(property "Description" ""
+		(property "Description" "Resistor, small symbol"
 			(at 31.75 64.77 0)
 			(effects
@@
 			)
 		)
-		(property "Description" ""
+		(property "Description" "Resistor, small symbol"
 			(at 54.61 64.77 0)
 			(effects
@@
 			)
 		)
-		(property "Description" ""
+		(property "Description" "Resistor, small symbol"
 			(at 39.37 64.77 0)
 			(effects
@@
 	)
 	(symbol
-		(lib_id "Symbols:DGND")
+		(lib_id "power:GNDD")
 		(at 185.42 59.69 0)
 		(unit 1)
@@
 			)
 		)
-		(property "Description" ""
+		(property "Description" "Power symbol creates a global label with name \"GNDD\" , digital ground"
 			(at 185.42 59.69 0)
 			(effects
@@
 			)
 		)
-		(property "Datasheet" "${KIPRJMOD}\\datasheet\\PYu_RT_1_to_0_01_RoHS_L_12-3003070.pdf"
+		(property "Datasheet" "~"
 			(at 142.24 85.09 0)
 			(effects
@@
 			)
 		)
-		(property "Description" ""
+		(property "Description" "Resistor, small symbol"
 			(at 142.24 85.09 0)
 			(effects
@@
 	)
 	(symbol
-		(lib_id "Symbols:DGND")
+		(lib_id "power:GNDD")
 		(at 170.18 81.28 0)
 		(unit 1)
@@
 			)
 		)
-		(property "Description" ""
+		(property "Description" "Power symbol creates a global label with name \"GNDD\" , digital ground"
 			(at 170.18 81.28 0)
 			(effects
@@
 			)
 		)
-		(property "Datasheet" "${KIPRJMOD}\\datasheet\\PYu_RT_1_to_0_01_RoHS_L_12-3003070.pdf"
+		(property "Datasheet" "~"
 			(at 170.18 88.9 0)
 			(effects
@@
 			)
 		)
-		(property "Description" ""
+		(property "Description" "Resistor, small symbol"
 			(at 170.18 88.9 0)
 			(effects
@@
 			)
 		)
-		(property "Description" ""
+		(property "Description" "Resistor, small symbol"
 			(at 46.99 64.77 0)
 			(effects
@@
 			)
 		)
-		(property "Description" ""
+		(property "Description" "Resistor, small symbol"
 			(at 68.58 68.58 0)
 			(effects
@@
 	)
 	(symbol
-		(lib_id "Symbols:DGND")
+		(lib_id "power:GNDD")
 		(at 118.11 85.09 0)
 		(unit 1)
@@
 			)
 		)
-		(property "Description" ""
+		(property "Description" "Power symbol creates a global label with name \"GNDD\" , digital ground"
 			(at 118.11 85.09 0)
 			(effects
@@
 			)
 		)
-		(property "Description" ""
+		(property "Description" "Resistor, small symbol"
 			(at 59.69 72.39 0)
 			(effects
@@
 	)
 	(symbol
-		(lib_id "Symbols:+12V_PGND")
+		(lib_id "power:+12V")
 		(at 85.09 45.72 0)
 		(unit 1)
 		(exclude_from_sim no)
-		(in_bom no)
-		(on_board no)
+		(in_bom yes)
+		(on_board yes)
 		(dnp no)
 		(fields_autoplaced yes)
@@
 		)
 		(property "Footprint" ""
-			(at 88.265 43.18 0)
+			(at 85.09 45.72 0)
 			(effects
 				(font
@@
 		)
 		(property "Datasheet" ""
-			(at 88.265 43.18 0)
-			(effects
-				(font
-					(size 1.27 1.27)
-				)
-				(hide yes)
-			)
-		)
-		(property "Description" ""
 			(at 85.09 45.72 0)
 			(effects
@@
 			)
 		)
+		(property "Description" "Power symbol creates a global label with name \"+12V\""
+			(at 85.09 45.72 0)
+			(effects
+				(font
+					(size 1.27 1.27)
+				)
+				(hide yes)
+			)
+		)
 		(pin "1"
 		)
@@
 	)
 	(symbol
-		(lib_name "R_Small_14")
 		(lib_id "Device:R_Small")
 		(at 128.27 69.85 90)
@@
 			)
 		)
-		(property "Datasheet" "${KIPRJMOD}\\datasheet\\PYu_RT_1_to_0_01_RoHS_L_12-3003070.pdf"
+		(property "Datasheet" "~"
 			(at 128.27 69.85 0)
 			(effects
@@
 			)
 		)
-		(property "Description" ""
+		(property "Description" "Resistor, small symbol"
 			(at 128.27 69.85 0)
 			(effects

Commit message: Tidied up the schematic. Added the pdf version for V0.9.
Signed-off-by: Jean Alinei <jean.alinei@owntech.org>
Other:
- title: Micro-inverter - 400W -> Grid voltage measurement
- moved on the sheet: C406, C407, C501, C502, C503, C505, R501, R502, R503, R504, Rv501, Rv502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
