File: KiCAD_Files/uVerter.kicad_sch (KiCad schematic)
At the start: 15 parts

Commit message: Tidied up the schematic. Added the pdf version for V0.9.
Signed-off-by: Jean Alinei <jean.alinei@owntech.org>
Parts:
- FID1, FID2, FID3, Logo1, N101: now fitted
Other:
- sheet Feeder renamed Internal power supplies
- sheet Power renamed Power stage
- sheet Signal Isolators renamed PWM Signal Isolators
- note added: "Net Ties"
- note added: "PCB screw mounts M3 Height 3.5mm"
- note added: "Thermal standoffs"
- note removed: "Do we need DCBus current ?"
- note removed: "Heatsinks HV switching nodes thermal standoffs"
- note removed: "Heatsinks LV switching nodes thermal standoffs"
- note removed: "Heatsinks diodes nodes thermal standoffs"
- note removed: "M3 Height 3.5mm"
- title: Micro-inverter - 400W -> Micro-inverter - 450W
- moved on the sheet: H1, H2, H3, H4, H5, H6, HS10, HS3, HS4, HS9
