File: KiCAD_Files/feeder.kicad_sch (KiCad schematic)
At the start: 50 parts, among them U702 TPS562202, U703 VPS8701B, U704 VPS8701B, U705 TL431, U707 LMR38020SDDAR

Commit message: Added LSW3 and LSW4 netclass (Fix #3). Tidied up courtyard DRC for testpoints.
Signed-off-by: Jean Alinei <jean.alinei@owntech.org>
Parts:
- TP701, TP702, TP703, TP704, TP705, TP706, TP707: footprint TestPoint:TestPoint_Pad_D1.0mm -> Footprints:TestPoint_Pad_D1.0mm
Changed lines of the file:
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@@
 			)
 		)
-		(property "Footprint" "TestPoint:TestPoint_Pad_D1.0mm"
+		(property "Footprint" "Footprints:TestPoint_Pad_D1.0mm"
 			(at 246.38 139.7 0)
 			(effects
@@
 			)
 		)
-		(property "Footprint" "TestPoint:TestPoint_Pad_D1.0mm"
+		(property "Footprint" "Footprints:TestPoint_Pad_D1.0mm"
 			(at 210.82 91.44 0)
 			(effects
@@
 			)
 		)
-		(property "Footprint" "TestPoint:TestPoint_Pad_D1.0mm"
+		(property "Footprint" "Footprints:TestPoint_Pad_D1.0mm"
 			(at 233.68 36.83 0)
 			(effects
@@
 			)
 		)
-		(property "Footprint" "TestPoint:TestPoint_Pad_D1.0mm"
+		(property "Footprint" "Footprints:TestPoint_Pad_D1.0mm"
 			(at 246.38 161.29 0)
 			(effects
@@
 			)
 		)
-		(property "Footprint" "TestPoint:TestPoint_Pad_D1.0mm"
+		(property "Footprint" "Footprints:TestPoint_Pad_D1.0mm"
 			(at 233.68 54.61 0)
 			(effects
@@
 			)
 		)
-		(property "Footprint" "TestPoint:TestPoint_Pad_D1.0mm"
+		(property "Footprint" "Footprints:TestPoint_Pad_D1.0mm"
 			(at 209.55 104.14 0)
 			(effects
@@
 			)
 		)
-		(property "Footprint" "TestPoint:TestPoint_Pad_D1.0mm"
+		(property "Footprint" "Footprints:TestPoint_Pad_D1.0mm"
 			(at 148.59 34.29 0)
 			(effects
