File: KiCAD_Files/power.kicad_sch (KiCad schematic)
At the start: 170 parts, among them J1 Conn_01x01, J2 Conn_01x01, J3 Conn_01x01, J5 Conn_01x01, J8 Conn_01x01, K1 HF140FF/012-2HSWTF, Q1 CID12N65D, Q10 CJAC90SN12, Q11 ZXMN7A11GTA, Q2 CID12N65D, Q3 CID12N65D, Q4 CID12N65D, Q5 CJAC90SN12, Q6 CJAC90SN12, Q7 CJAC90SN12, Q8 CJAC90SN12, Q9 CJAC90SN12, T1 Transformer_1P_1S, T2 Transformer_1P_1S, U1 INA240A1PWR, U2 INA240A1PWR, U3 UCC27282DRC, U4 UCC27282DRC

Commit message: Tidied up the schematic. Added the pdf version for V0.9.
Signed-off-by: Jean Alinei <jean.alinei@owntech.org>
Parts:
- Logo101: now fitted
Other:
- title: (none) -> Power stage
- moved on the sheet: HS101, HS104, HS105, HS106, HS107, HS108, HS109, HS11, HS110, HS111, HS12, HS5

Commit message: Modified the differential inductor filter footprints slightly. Solves #2.
Signed-off-by: Jean Alinei <jean.alinei@owntech.org>
Parts:
- L1, L3: footprint Footprints:L_SMD_L27.0-W19.5-LS23.5_60B104C -> Footprints:L_SMD_L28.0-W23-LS25
Changed lines of the file:
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@@
 			)
 		)
-		(property "Footprint" "Footprints:L_SMD_L27.0-W19.5-LS23.5_60B104C"
+		(property "Footprint" "Footprints:L_SMD_L28.0-W23-LS25"
 			(at 213.36 73.66 0)
 			(effects
@@
 			)
 		)
-		(property "Footprint" "Footprints:L_SMD_L27.0-W19.5-LS23.5_60B104C"
+		(property "Footprint" "Footprints:L_SMD_L28.0-W23-LS25"
 			(at 213.36 55.88 0)
 			(effects

Commit message: Added LSW3 and LSW4 netclass (Fix #3). Tidied up courtyard DRC for testpoints.
Signed-off-by: Jean Alinei <jean.alinei@owntech.org>
Parts:
- TP101, TP103, TP105, TP107: footprint TestPoint:TestPoint_Pad_D1.0mm -> Footprints:TestPoint_Pad_D0.5mm
- TP102, TP104, TP106, TP108, TP109: footprint TestPoint:TestPoint_Pad_D1.0mm -> Footprints:TestPoint_Pad_D1.0mm
Changed lines of the file:
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@@
 			)
 		)
-		(property "Footprint" "TestPoint:TestPoint_Pad_D1.0mm"
+		(property "Footprint" "Footprints:TestPoint_Pad_D0.5mm"
 			(at 193.04 234.95 0)
 			(effects
@@
 			)
 		)
-		(property "Footprint" "TestPoint:TestPoint_Pad_D1.0mm"
+		(property "Footprint" "Footprints:TestPoint_Pad_D1.0mm"
 			(at 167.64 184.15 0)
 			(effects
@@
 			)
 		)
-		(property "Footprint" "TestPoint:TestPoint_Pad_D1.0mm"
+		(property "Footprint" "Footprints:TestPoint_Pad_D0.5mm"
 			(at 180.34 199.39 0)
 			(effects
@@
 			)
 		)
-		(property "Footprint" "TestPoint:TestPoint_Pad_D1.0mm"
+		(property "Footprint" "Footprints:TestPoint_Pad_D1.0mm"
 			(at 300.99 17.78 0)
 			(effects
@@
 			)
 		)
-		(property "Footprint" "TestPoint:TestPoint_Pad_D1.0mm"
+		(property "Footprint" "Footprints:TestPoint_Pad_D1.0mm"
 			(at 180.34 214.63 0)
 			(effects
@@
 			)
 		)
-		(property "Footprint" "TestPoint:TestPoint_Pad_D1.0mm"
+		(property "Footprint" "Footprints:TestPoint_Pad_D0.5mm"
 			(at 181.61 132.08 0)
 			(effects
@@
 			)
 		)
-		(property "Footprint" "TestPoint:TestPoint_Pad_D1.0mm"
+		(property "Footprint" "Footprints:TestPoint_Pad_D1.0mm"
 			(at 162.56 251.46 0)
 			(effects
@@
 			)
 		)
-		(property "Footprint" "TestPoint:TestPoint_Pad_D1.0mm"
+		(property "Footprint" "Footprints:TestPoint_Pad_D0.5mm"
 			(at 167.64 166.37 0)
 			(effects
@@
 			)
 		)
-		(property "Footprint" "TestPoint:TestPoint_Pad_D1.0mm"
+		(property "Footprint" "Footprints:TestPoint_Pad_D1.0mm"
 			(at 181.61 147.32 0)
 			(effects
